File: hardware/kicad/ipod-hat.kicad_pcb (KiCad board)
At the start: 2 copper layers, 65 x 56.5 mm, 4 parts

Commit message: Add documentation, LICENSE, and rename project to ownPod
Co-Authored-By: Claude Sonnet 4.6 <noreply@anthropic.com>
Other:
- board text added: "ownPod HAT v0.1"
- board text removed: "iPod Player HAT v0.1"
Changed lines of the file:
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@@
   )
   ;; Silkscreen labels for component placement zones
-  (gr_text "iPod Player HAT v0.1" (at 32.5 54) (layer "F.SilkS")
+  (gr_text "ownPod HAT v0.1" (at 32.5 54) (layer "F.SilkS")
     (effects (font (size 1.5 1.5) (thickness 0.15)))
 )
