File: hardware/kicad/ipod-hat.kicad_sch (KiCad schematic)
At the start: 39 parts, among them J1 RPi_GPIO_Header, J2 3.5mm_Jack, J3 USB-C, J4 LiPo_JST, J5 ST7789_Display, SW1 PWR_SW, SW2 Encoder, SW3 MENU, SW4 BACK, SW5 PLAY, U1 PCM5102A, U2 TP4056, U3 MT3608

Commit message: Add documentation, LICENSE, and rename project to ownPod
Co-Authored-By: Claude Sonnet 4.6 <noreply@anthropic.com>
Other:
- title: iPod Player HAT -> ownPod HAT
Changed lines of the file:
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@@
   (paper "A3")
   (title_block
-    (title "iPod Player HAT")
+    (title "ownPod HAT")
     (date "2026-06-18")
     (rev "0.1")
